Commit message: floor moveit config

File: src/abb_linear_axis_floor/urdf/abb_linear_axis_floor.urdf (robot description, URDF)
Before this commit: robot linear_axis_two_robots, 22 links, 21 joints
Links:
- link axis: geometry collision mesh filename=package://abb_linear_axis_floor/meshes/collision/axis_floor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; visual mesh filename=package://abb_linear_axis_floor/meshes/visual/axis_floor.stl
- link cartA: geometry collision mesh filename=package://abb_linear_axis_floor/meshes/collision/cart_floor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; visual mesh filename=package://abb_linear_axis_floor/meshes/visual/cart_floor.stl
- link cartB: geometry collision mesh filename=package://abb_linear_axis_floor/meshes/collision/cart_floor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; visual mesh filename=package://abb_linear_axis_floor/meshes/visual/cart_floor.stl
