Commit message: overhead side

File: src/abb_linear_axis_overhead_side/urdf/abb_linear_axis_overhead_side.urdf (robot description, URDF)
Before this commit: robot linear_axis_two_robots, 22 links, 21 joints
Links:
- link axis: geometry collision mesh filename=package://abb_linear_axis_overhead_side/meshes/collision/ax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; visual mesh filename=package://abb_linear_axis_overhead_side/meshes/visual/axis_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
- link cartA: geometry collision mesh filename=package://abb_linear_axis_overhead_side/meshes/collision/ca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; visual mesh filename=package://abb_linear_axis_overhead_side/meshes/visual/cart_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
- link cartB: geometry collision mesh filename=package://abb_linear_axis_overhead_side/meshes/collision/ca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; visual mesh filename=package://abb_linear_axis_overhead_side/meshes/visual/cart_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
